Commit message: correct call for leorover zed camera

File: gazebo-simulator/rovers/leorover/leo_erc_description/urdf/leo_erc.xacro (robot description, xacro)
@@ -1,4 +1,7 @@
 <?xml version="1.0" encoding="utf-8"?>
 <robot xmlns:xacro="http://www.ros.org/wiki/xacro">
+  <!--##########-->
+  <!-- LEO ERC -->
+  <!--##########-->
   <xacro:macro name="leo_erc"
                params="default_antenna:=true
@@ -93,5 +96,5 @@
       </link>
     </xacro:macro>
-    <!-- LINKS -->
+    <!-- links -->
     <xacro:if value="${footprint_link}">
       <link name="${link_prefix}base_footprint"/>
@@ -263,5 +266,7 @@
     </joint>
   </xacro:macro>
+  <!--##########-->
   <!-- LEO GAZEBO -->
+  <!--##########-->
   <xacro:macro name="leo_gazebo"
                params="robot_ns:='''">
@@ -421,5 +426,5 @@
       </collision>
     </gazebo>
-    <!-- camera -->
+    <!-- Leo camera -->
     <gazebo reference="${link_prefix}camera_frame">
       <sensor name="camera" type="camera">
@@ -471,4 +476,5 @@
       </plugin>
     </gazebo>
+    <!-- Leo IMU -->
     <gazebo reference="${link_prefix}imu_frame">
       <sensor type="imu" name="leo_imu_sensor">
@@ -503,4 +509,7 @@
     </gazebo>
   </xacro:macro>
+  <!--##########-->
+  <!--  LEO SIM -->
+  <!--##########-->
   <xacro:macro name="leo_sim"
                params="default_antenna:=true
@@ -526,6 +535,8 @@
     </xacro:if>
   </xacro:macro>
-  <xacro:include filename="$(find leo_erc_description)/urdf/zed2.xacro"/>
-  <xacro:macro name="zed2_gazebo"
+  <!--##########-->
+  <!-- ZED2 GAZEBO-->
+  <!--##########-->
+  <xacro:macro name="zed2_leo_gazebo"
                params="default_antenna:=true
                        robot_ns:=''
@@ -536,64 +547,69 @@
                        imu_translation:='0.0628 -0.0314 -0.0393'
                        mecanum_wheels:=false">
-  <joint name="${joint_prefix}erc_payload_joint" type="fixed">
-    <origin xyz="0 0 0" rpy="0 0 0"/>
-    <parent link="${link_prefix}base_link"/>
-    <child link="${link_prefix}erc_payload_link"/>
-  </joint>
-  <link name="${link_prefix}erc_payload_link">
-    <inertial>
-      <mass value="1.33042"/>
-      <origin xyz="-0.055949 0.001702 0.064261"/>
-      <inertia
-        ixx="0.007414" ixy="0.00007852" ixz="-0.003995"
-        iyy="0.01745" iyz="-0.00001858"
-        izz="0.01187"/>
-    </inertial>
-    <visual>
-      <geometry>
-        <mesh filename="package://leo_description/models/ERC2021payload.dae"/>
-      </geometry>
-    </visual>
-    <collision>
-      <geometry>
-        <mesh filename="package://leo_description/models/ERC2021payload_outline.dae"/>
-      </geometry>
-    </collision>
-  </link>
-  <joint name="${joint_prefix}zed2_tilt_head_joint" type="fixed">
-    <origin xyz="0.048 0 0.141" rpy="0 0.415911961 0"/> <!-- 23.83 degree tilt -->
-    <parent link="${link_prefix}erc_payload_link"/>
-    <child link="${link_prefix}zed2_tilt_head_link"/>
-  </joint>
-  <link name="${link_prefix}zed2_tilt_head_link">
-    <inertial>
-      <mass value="0.108614"/>
-      <origin xyz="0 -0.008564 0.015313"/>
-      <inertia
-        ixx="7.371e-5" ixy="0.0" ixz="1.326071e-6"
-        iyy="3.14e-5" iyz="-1.424e-5"
-        izz="6.13e-5"/>
-    </inertial>
-    <visual>
-      <origin xyz="0 0 0" rpy="0 0 ${pi}"/>
-      <geometry>
-        <mesh filename="package://leo_description/models/Manfrotto_head.dae"/>
-      </geometry>
-    </visual>
-    <collision>
-      <origin xyz="0 0 0" rpy="0 0 ${pi}"/>
-      <geometry>
-        <mesh filename="package://leo_description/models/Manfrotto_head.dae"/>
-      </geometry>
-    </collision>
-  </link>
-  <joint name="${joint_prefix}zed2_camera_center_joint" type="fixed">
-    <parent link="${link_prefix}zed2_tilt_head_link"/>
-    <child link="${link_prefix}zed2_camera_center"/>
-    <origin xyz="0 0 0.0486" rpy="0 0.032637657 0"/>
-  </joint>
-  <xacro:zed2 link_prefix="${link_prefix}"
-              joint_prefix="${joint_prefix}"/>
- </xacro:macro>
+    <joint name="${joint_prefix}erc_payload_joint" type="fixed">
+      <origin xyz="0 0 0" rpy="0 0 0"/>
+      <parent link="${link_prefix}base_link"/>
+      <child link="${link_prefix}erc_payload_link"/>
+    </joint>
+    <link name="${link_prefix}erc_payload_link">
+      <inertial>
+        <mass value="1.33042"/>
+        <origin xyz="-0.055949 0.001702 0.064261"/>
+        <inertia
+          ixx="0.007414" ixy="0.00007852" ixz="-0.003995"
+          iyy="0.01745" iyz="-0.00001858"
+          izz="0.01187"/>
+      </inertial>
+      <visual>
+        <geometry>
+          <mesh filename="package://leo_description/models/ERC2021payload.dae"/>
+        </geometry>
+      </visual>
+      <collision>
+        <geometry>
+          <mesh filename="package://leo_description/models/ERC2021payload_outline.dae"/>
+        </geometry>
+      </collision>
+    </link>
+    <joint name="${joint_prefix}zed2_tilt_head_joint" type="fixed">
+      <origin xyz="0.048 0 0.141" rpy="0 0.415911961 0"/> <!-- 23.83 degree tilt -->
+      <parent link="${link_prefix}erc_payload_link"/>
+      <child link="${link_prefix}zed2_tilt_head_link"/>
+    </joint>
+    <link name="${link_prefix}zed2_tilt_head_link">
+      <inertial>
+        <mass value="0.108614"/>
+        <origin xyz="0 -0.008564 0.015313"/>
+        <inertia
+          ixx="7.371e-5" ixy="0.0" ixz="1.326071e-6"
+          iyy="3.14e-5" iyz="-1.424e-5"
+          izz="6.13e-5"/>
+      </inertial>
+      <visual>
+        <origin xyz="0 0 0" rpy="0 0 ${pi}"/>
+        <geometry>
+          <mesh filename="package://leo_description/models/Manfrotto_head.dae"/>
+        </geometry>
+      </visual>
+      <collision>
+        <origin xyz="0 0 0" rpy="0 0 ${pi}"/>
+        <geometry>
+          <mesh filename="package://leo_description/models/Manfrotto_head.dae"/>
+        </geometry>
+      </collision>
+    </link>
+    <joint name="${joint_prefix}zed2_camera_center_joint" type="fixed">
+      <parent link="${link_prefix}zed2_tilt_head_link"/>
+      <child link="${link_prefix}zed2_camera_center"/>
+      <origin xyz="0 0 0.0486" rpy="0 0.032637657 0"/>
+    </joint>
+    <xacro:zed2 link_prefix="${link_prefix}"
+                joint_prefix="${joint_prefix}"/>
+    <xacro:zed2_gazebo link_prefix="${link_prefix}"
+                joint_prefix="${joint_prefix}"/>
+  </xacro:macro>
+  <!--##########-->
+  <!--  LEO ERC GAZEBO -->
+  <!--##########-->
   <xacro:macro name="leo_erc_gazebo"
                params="robot_ns:=''">
@@ -603,5 +619,4 @@
     </xacro:if>
     <xacro:leo_gazebo robot_ns="${robot_ns}"/>
-    <xacro:zed2_gazebo robot_ns="${robot_ns}"/>
     <gazebo>
       <plugin
@@ -612,4 +627,7 @@
     </gazebo>
   </xacro:macro>
+  <!--##########-->
+  <!--  LEO ERC SIM -->
+  <!--##########-->
   <xacro:macro name="leo_erc_sim"
                params="default_antenna:=true

File: gazebo-simulator/rovers/leorover/leo_erc_description/urdf/leo_erc_sim.urdf.xacro (robot description, xacro)
@@ -6,6 +6,8 @@
   <xacro:arg name="mecanum_wheels" default="false"/>
   <xacro:include filename="$(find leo_erc_description)/urdf/leo_erc.xacro"/>
+  <xacro:include filename="$(find leo_erc_description)/urdf/zed2.xacro"/>
   <xacro:leo_erc_sim robot_ns="$(arg robot_ns)"
                      fixed="$(arg fixed)"
                      mecanum_wheels="$(arg mecanum_wheels)"/>
+  <xacro:zed2_leo_gazebo/>
 </robot>

File: gazebo-simulator/rovers/leorover/leo_erc_description/urdf/zed2.xacro (robot description, xacro)
@@ -2,4 +2,7 @@
 <robot xmlns:xacro="http://ros.org/wiki/xacro">
   <xacro:property name="baseline" value="0.12"/>
+ <!--##########-->
+ <!--  ZED2 -->
+ <!--##########-->
   <xacro:macro name="zed2"
                params="link_prefix:=''
@@ -78,6 +81,16 @@
     <link name="${link_prefix}zed2_temp_right_link" />
   </xacro:macro>
+ <!--##########-->
+ <!--  ZED2 GAZEBO -->
+ <!--##########-->
   <xacro:macro name="zed2_gazebo"
-               params="robot_ns:=''">
+               params="default_antenna:=true
+                       robot_ns:=''
+                       rockers_fixed:=true
+                       footprint_link:=true
+                       link_prefix:=''
+                       joint_prefix:=''
+                       imu_translation:='0.0628 -0.0314 -0.0393'
+                       mecanum_wheels:=false">
     <xacro:property name="link_prefix" value=""/>
     <xacro:if value="${robot_ns != '' and robot_ns != '/'}">
@@ -87,8 +100,8 @@
     <gazebo reference="${link_prefix}zed2_left_camera_frame">
       <sensor type="imu" name="zed2_imu_sensor">
-        <always_on>true</always_on>
-        <update_rate>50</update_rate>
+        <update_rate>100</update_rate>
         <visualize>true</visualize>
         <topic>${link_prefix}zed2/imu/data</topic>
+        <always_on>1</always_on>
         <gz_frame_id>${link_prefix}zed2_left_camera_frame</gz_frame_id>
       </sensor>
@@ -155,45 +168,29 @@
         <gz_frame_id>${link_prefix}zed2_left_camera_frame</gz_frame_id>
       </sensor>
-      <sensor type="depth" name="zed2_depth_camera">
+      <sensor type="depth_camera" name="zed2_depth_camera">
         <!-- Rectified images, Depth images, Point Clouds -->
-        <always_on>true</always_on>
-        <update_rate>15.0</update_rate>
+        <always_on>1</always_on>
+        <update_rate>15</update_rate>
         <visualize>true</visualize>
         <camera name="zed2_depth">
-          <horizontal_fov>1.7633</horizontal_fov>
-          <image>
-            <width>1280</width>
-            <height>720</height>
-            <format>R8G8B8</format>
-          </image>
-          <clip>
-            <near>0.02</near>
-            <far>300</far>
-          </clip>
-          <noise>
-            <type>gaussian</type>
-            <mean>0.0</mean>
-            <stddev>0.007</stddev>
+          <horizontal_fov>1.274</horizontal_fov>
+          <image>
+            <width>640</width>
+            <height>480</height>
+            <format>R_FLOAT32</format>
+          </image>
+          <clip>
+            <near>0.1</near>
+            <far>20</far>
+          </clip>
+          <noise>
+            <type>gaussian</type>
+            <mean>0.0</mean>
+            <stddev>0.01</stddev>
           </noise>
         </camera>
         <topic>${link_prefix}zed2/depth</topic>
-        <gz_frame_id>${link_prefix}zed2_left_camera_frame</gz_frame_id>
-        <!-- <plugin name="camera_controller" filename="libgazebo_ros_openni_kinect.so">
-          <robotNamespace>${robot_ns}</robotNamespace>
-          <cameraName>zed2</cameraName>
-          <imageTopicName>left/image_rect_color</imageTopicName>
-          <cameraInfoTopicName>left/camera_info</cameraInfoTopicName>
-          <depthImageTopicName>depth/depth_registered</depthImageTopicName>
-          <depthImageInfoTopicName>depth/camera_info</depthImageInfoTopicName>
-          <pointCloudTopicName>point_cloud/cloud_registered</pointCloudTopicName>
-          <pointCloudCutoff>0.3</pointCloudCutoff>
-          <pointCloudCutoffMax>20.0</pointCloudCutoffMax>
-          <frameName>zed2_left_camera_optical_frame</frameName>
-          <baseline>0.12</baseline>
-          <CxPrime>658.8206787109375</CxPrime>
-          <Cx>658.8206787109375</Cx>
-          <Cy>372.25787353515625</Cy>
-          <hackBaseline>0.0</hackBaseline>
-        </plugin> -->
+        <pointCloudTopicName>${link_prefix}zed2/depth/points</pointCloudTopicName>
+        <gz_frame_id>${link_prefix}zed2_left_camera_frame</gz_frame_id>
       </sensor>
     </gazebo>
