Commit message: remove ERC, add ouster and zed and simplify packages

File: gazebo-simulator/rovers/leorover/leo_description/urdf/leo_sim.urdf.xacro (robot description, xacro)
@@ -6,4 +6,12 @@
   <xacro:arg name="mecanum_wheels" default="false"/>
   <xacro:include filename="$(find leo_description)/urdf/macros.xacro"/>
+  <xacro:include filename="$(find ouster_description)/urdf/OS1-64.urdf.xacro"/>
+  <xacro:include filename="$(find zed2_description)/urdf/zed2.urdf.xacro"/>
+  <xacro:OS1-64 name="os1_sensor" hz="10" samples="220">
+    <origin xyz="0 0 0.25" rpy="0 0 0" />
+  </xacro:OS1-64>
+  <xacro:Zed2 name="zed2" >
+    <origin xyz="0.048 0 0.101" rpy="0 0.415911961 0"/>
+  </xacro:Zed2>
   <xacro:leo_sim robot_ns="$(arg robot_ns)"
                  fixed="$(arg fixed)"

File: gazebo-simulator/rovers/leorover/leo_description/urdf/macros.xacro (robot description, xacro)
@@ -348,5 +348,5 @@
               <mu>1</mu>
               <mu2>1</mu2>
-              <slip1>0.035</slip1>
+              <slip1>0.0035</slip1>
               <slip2>0</slip2>
               <fdir1>0 0 1</fdir1>
@@ -368,5 +368,5 @@
               <mu>1</mu>
               <mu2>1</mu2>
-              <slip1>0.035</slip1>
+              <slip1>0.0035</slip1>
               <slip2>0</slip2>
               <fdir1>0 0 1</fdir1>
@@ -388,5 +388,5 @@
               <mu>1</mu>
               <mu2>1</mu2>
-              <slip1>0.035</slip1>
+              <slip1>0.0035</slip1>
               <slip2>0</slip2>
               <fdir1>0 0 1</fdir1>
@@ -408,5 +408,5 @@
               <mu>1</mu>
               <mu2>1</mu2>
-              <slip1>0.035</slip1>
+              <slip1>0.0035</slip1>
               <slip2>0</slip2>
               <fdir1>0 0 1</fdir1>
@@ -432,5 +432,5 @@
               </image>
               <clip>
-                  <near>0.2</near>
+                  <near>0.1</near>
                   <far>300</far>
               </clip>

File: gazebo-simulator/rovers/scout_agilex/scout_description/urdf/scout_wheel_type1.xacro (robot description, xacro)
@@ -49,9 +49,10 @@
             </collision>
         </link>
-        <joint name="${wheel_prefix}_wheel" type="continuous">
+        <joint name="${wheel_prefix}_wheel" type="revolute">
             <parent link="base_link"/>
             <child link="${wheel_prefix}_wheel_link"/>
             <xacro:insert_block name="joint_pose"/>
             <axis xyz="0 -1 0" rpy="0 0 0" />
+            <limit effort="5" velocity="6.28"  lower="-1.79769e+308" upper="1.79769e+308" />
             <dynamics damping="0.0" friction="20"/>
         </joint>

File: gazebo-simulator/rovers/scout_agilex/scout_description/urdf/scout_wheel_type2.xacro (robot description, xacro)
@@ -49,9 +49,10 @@
             </collision>
         </link>
-        <joint name="${wheel_prefix}_wheel" type="continuous">
+        <joint name="${wheel_prefix}_wheel" type="revolute">
             <parent link="base_link"/>
             <child link="${wheel_prefix}_wheel_link"/>
             <xacro:insert_block name="joint_pose"/>
             <axis xyz="0 -1 0" rpy="0 0 0" />
+            <limit effort="5" velocity="6.28"  lower="-1.79769e+308" upper="1.79769e+308" />
             <dynamics damping="0.0" friction="20"/>
         </joint>
